File: PCB_Glove.kicad_pcb (KiCad board)
At the start: 4 copper layers, 50 x 64.5 mm, 12 parts, among them J1 HC-05, J2 MPU-9250/6500, J4 MPU-9250/6500, J5 FlexSensor_JST, J6 External_source, SW1 SW_SPST, SW2 SW_SPST, SW3 SW_SPST

Commit message: changes in pcb
Other:
- board text added: "King of the castle King of the castle"
- board text added: "Made by Johnan Luca Last mod: 16/12/2025"
Changed lines of the file:
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@@
 		(layer "Edge.Cuts")
 	)
-	(gr_text "-"
+	(gr_text "Made by Johnan Luca\nLast mod: 16/12/2025\n"
+		(at 123.5 95 0)
+		(layer "F.SilkS")
+		(effects
+			(font
+				(size 0.8 0.8)
+				(thickness 0.1)
+			)
+			(justify left)
+		)
+	)
+	(gr_text "+\n"
 		(at 132 104 0)
 		(layer "F.SilkS")
@@
 				(thickness 0.2)
 				(bold yes)
+			)
+			(justify left bottom)
+		)
+	)
+	(gr_text "King of the castle\n	King of the castle"
+		(at 150 103 90)
+		(layer "F.SilkS")
+		(effects
+			(font
+				(size 1 1)
+				(thickness 0.1)
 			)
 			(justify left bottom)
@@
 		)
 	)
-	(gr_text "+"
-		(at 132 112.5 0)
+	(gr_text "-\n"
+		(at 133 112.5 90)
 		(layer "F.SilkS")
 		(effects
