File: PCB_Glove.kicad_pcb (KiCad board)
At the start: 4 copper layers, 50 x 64.5 mm, 12 parts, among them J1 HC-05, J2 MPU-9250/6500, J4 MPU-9250/6500, J5 FlexSensor_JST, J6 External_source, SW1 SW_SPST, SW2 SW_SPST, SW3 SW_SPST

Commit message: Polished Schematic
Connections:
- net Net-(A1-+5V) renamed /+5V
- net Net-(A1-3V3) renamed /+3V3
- net Net-(A1-A0) renamed /A0
- net Net-(A1-D2) renamed /INT1
- net Net-(A1-D3) renamed /INT2
- net Net-(A1-SCL/A5) renamed /SCL
- net Net-(A1-SDA/A4) renamed /SDA
- net VCC renamed +9V
Changed lines of the file:
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@@
 	(net 3 "unconnected-(A1-~{RESET}-Pad3)")
 	(net 4 "unconnected-(A1-SCK-Pad16)")
-	(net 5 "Net-(A1-SDA{slash}A4)")
-	(net 6 "Net-(A1-D3)")
+	(net 5 "/SDA")
+	(net 6 "/INT2")
 	(net 7 "unconnected-(A1-A6-Pad25)")
 	(net 8 "unconnected-(A1-D7-Pad10)")
-	(net 9 "Net-(A1-D2)")
+	(net 9 "/INT1")
 	(net 10 "unconnected-(A1-D8-Pad11)")
 	(net 11 "Net-(A1-RX1)")
 	(net 12 "unconnected-(A1-A1-Pad20)")
-	(net 13 "Net-(A1-3V3)")
+	(net 13 "/+5V")
 	(net 14 "unconnected-(A1-A7-Pad26)")
 	(net 15 "unconnected-(A1-~{RESET}-Pad28)")
@@
 	(net 21 "unconnected-(A1-D6-Pad9)")
 	(net 22 "unconnected-(A1-D5-Pad8)")
-	(net 23 "Net-(A1-SCL{slash}A5)")
-	(net 24 "Net-(A1-+5V)")
+	(net 23 "/+3V3")
+	(net 24 "/SCL")
 	(net 25 "unconnected-(A1-A2-Pad21)")
 	(net 26 "Net-(A1-TX1)")
@@
 	(net 34 "unconnected-(J2-Pin_5-Pad5)")
 	(net 35 "Net-(A1-VIN)")
-	(net 36 "Net-(A1-A0)")
+	(net 36 "/A0")
 	(net 37 "Net-(J1-Pin_2)")
 	(net 38 "unconnected-(J4-Pin_5-Pad5)")
@@
 	(net 42 "GND")
 	(net 43 "Net-(SW2-A)")
-	(net 44 "VCC")
+	(net 44 "+9V")
 	(footprint "Connector_JST:JST_PH_B2B-PH-K_1x02_P2.00mm_Vertical"
 		(layer "F.Cu")
@@
 			(remove_unused_layers no)
 			(roundrect_rratio 0.208333)
-			(net 36 "Net-(A1-A0)")
+			(net 36 "/A0")
 			(pinfunction "Pin_1")
 			(pintype "passive")
@@
 			(layers "*.Cu" "*.Mask")
 			(remove_unused_layers no)
-			(net 24 "Net-(A1-+5V)")
+			(net 13 "/+5V")
 			(pinfunction "Pin_2")
 			(pintype "passive")
@@
 			(layers "*.Cu" "*.Mask")
 			(remove_unused_layers no)
-			(net 24 "Net-(A1-+5V)")
+			(net 13 "/+5V")
 			(pinfunction "Pin_1")
 			(pintype "passive")
@@
 			(layers "*.Cu" "*.Mask")
 			(remove_unused_layers no)
-			(net 23 "Net-(A1-SCL{slash}A5)")
+			(net 24 "/SCL")
 			(pinfunction "Pin_3")
 			(pintype "passive")
@@
 			(layers "*.Cu" "*.Mask")
 			(remove_unused_layers no)
-			(net 5 "Net-(A1-SDA{slash}A4)")
+			(net 5 "/SDA")
 			(pinfunction "Pin_4")
 			(pintype "passive")
@@
 			(layers "*.Cu" "*.Mask")
 			(remove_unused_layers no)
-			(net 13 "Net-(A1-3V3)")
+			(net 23 "/+3V3")
 			(pinfunction "Pin_7")
 			(pintype "passive")
@@
 			(layers "*.Cu" "*.Mask")
 			(remove_unused_layers no)
-			(net 6 "Net-(A1-D3)")
+			(net 6 "/INT2")
 			(pinfunction "Pin_8")
 			(pintype "passive")
@@
 			(layers "F.Cu" "F.Mask" "F.Paste")
 			(roundrect_rratio 0.25)
-			(net 36 "Net-(A1-A0)")
+			(net 36 "/A0")
 			(pintype "passive")
 		)
@@
 			(layers "*.Cu" "*.Mask")
 			(remove_unused_layers no)
-			(net 24 "Net-(A1-+5V)")
+			(net 13 "/+5V")
 			(pinfunction "Pin_5")
 			(pintype "passive")
@@
 			(layers "*.Cu" "*.Mask")
 			(remove_unused_layers no)
-			(net 24 "Net-(A1-+5V)")
+			(net 13 "/+5V")
 			(pinfunction "Pin_1")
 			(pintype "passive")
@@
 			(layers "*.Cu" "*.Mask")
 			(remove_unused_layers no)
-			(net 23 "Net-(A1-SCL{slash}A5)")
+			(net 24 "/SCL")
 			(pinfunction "Pin_3")
 			(pintype "passive")
@@
 			(layers "*.Cu" "*.Mask")
 			(remove_unused_layers no)
-			(net 5 "Net-(A1-SDA{slash}A4)")
+			(net 5 "/SDA")
 			(pinfunction "Pin_4")
 			(pintype "passive")
@@
 			(layers "*.Cu" "*.Mask")
 			(remove_unused_layers no)
-			(net 9 "Net-(A1-D2)")
+			(net 9 "/INT1")
 			(pinfunction "Pin_8")
 			(pintype "passive")
@@
 			(remove_unused_layers no)
 			(roundrect_rratio 0.15625)
-			(net 44 "VCC")
+			(net 44 "+9V")
 			(pinfunction "A")
 			(pintype "passive")
@@
 			(remove_unused_layers no)
 			(roundrect_rratio 0.208333)
-			(net 44 "VCC")
+			(net 44 "+9V")
 			(pinfunction "Pin_1")
 			(pintype "passive")
@@
 			(layers "*.Cu" "*.Mask")
 			(remove_unused_layers no)
-			(net 9 "Net-(A1-D2)")
+			(net 9 "/INT1")
 			(pinfunction "D2")
 			(pintype "bidirectional")
@@
 			(layers "*.Cu" "*.Mask")
 			(remove_unused_layers no)
-			(net 6 "Net-(A1-D3)")
+			(net 6 "/INT2")
 			(pinfunction "D3")
 			(pintype "bidirectional")
@@
 			(layers "*.Cu" "*.Mask")
 			(remove_unused_layers no)
-			(net 13 "Net-(A1-3V3)")
+			(net 23 "/+3V3")
 			(pinfunction "3V3")
 			(pintype "power_out")
@@
 			(layers "*.Cu" "*.Mask")
 			(remove_unused_layers no)
-			(net 36 "Net-(A1-A0)")
+			(net 36 "/A0")
 			(pinfunction "A0")
 			(pintype "bidirectional")
@@
 			(layers "*.Cu" "*.Mask")
 			(remove_unused_layers no)
-			(net 5 "Net-(A1-SDA{slash}A4)")
+			(net 5 "/SDA")
 			(pinfunction "SDA/A4")
 			(pintype "bidirectional")
@@
 			(layers "*.Cu" "*.Mask")
 			(remove_unused_layers no)
-			(net 23 "Net-(A1-SCL{slash}A5)")
+			(net 24 "/SCL")
 			(pinfunction "SCL/A5")
 			(pintype "bidirectional")
@@
 			(layers "*.Cu" "*.Mask")
 			(remove_unused_layers no)
-			(net 24 "Net-(A1-+5V)")
+			(net 13 "/+5V")
 			(pinfunction "+5V")
 			(pintype "power_out")
@@
 	)
 	(segment
-		(start 163.1 111.4)
-		(end 163.5 111)
-		(width 0.2)
-		(layer "B.Cu")
-		(net 13)
-	)
-	(segment
-		(start 157.24 111.4)
-		(end 163.1 111.4)
-		(width 0.2)
-		(layer "B.Cu")
-		(net 13)
-	)
-	(segment
-		(start 159 73.975)
-		(end 163.475 69.5)
-		(width 0.2)
-		(layer "F.Cu")
-		(net 23)
-	)
-	(segment
-		(start 157.24 93.62)
-		(end 159 91.86)
-		(width 0.2)
-		(layer "F.Cu")
-		(net 23)
-	)
-	(segment
-		(start 159 91.86)
-		(end 159 73.975)
-		(width 0.2)
-		(layer "F.Cu")
-		(net 23)
-	)
-	(segment
-		(start 157.24 93.62)
-		(end 160.5 96.88)
-		(width 0.2)
-		(layer "B.Cu")
-		(net 23)
-	)
-	(segment
-		(start 160.5 96.88)
-		(end 160.5 97.84)
-		(width 0.2)
-		(layer "B.Cu")
-		(net 23)
-	)
-	(segment
-		(start 160.5 97.84)
-		(end 163.5 100.84)
-		(width 0.2)
-		(layer "B.Cu")
-		(net 23)
-	)
-	(segment
 		(start 117.5 79.5)
 		(end 118.16 78.84)
 		(width 0.2)
 		(layer "In2.Cu")
-		(net 24)
+		(net 13)
 	)
 	(segment
@@
 		(width 0.2)
 		(layer "In2.Cu")
-		(net 24)
+		(net 13)
 	)
 	(segment
@@
 		(width 0.2)
 		(layer "In2.Cu")
-		(net 24)
+		(net 13)
 	)
 	(segment
@@
 		(width 0.2)
 		(layer "In2.Cu")
-		(net 24)
+		(net 13)
 	)
 	(segment
@@
 		(width 0.2)
 		(layer "In2.Cu")
-		(net 24)
+		(net 13)
 	)
 	(segment
@@
 		(width 0.2)
 		(layer "In2.Cu")
-		(net 24)
+		(net 13)
 	)
 	(segment
@@
 		(width 0.2)
 		(layer "In2.Cu")
-		(net 24)
+		(net 13)
 	)
 	(segment
@@
 		(width 0.2)
 		(layer "In2.Cu")
-		(net 24)
+		(net 13)
 	)
 	(segment
@@
 		(width 0.2)
 		(layer "In2.Cu")
-		(net 24)
+		(net 13)
 	)
 	(segment
@@
 		(width 0.2)
 		(layer "In2.Cu")
-		(net 24)
+		(net 13)
 	)
 	(segment
@@
 		(width 0.2)
 		(layer "In2.Cu")
-		(net 24)
+		(net 13)
 	)
 	(segment
@@
 		(width 0.2)
 		(layer "In2.Cu")
-		(net 24)
+		(net 13)
 	)
 	(segment
@@
 		(width 0.2)
 		(layer "In2.Cu")
-		(net 24)
+		(net 13)
 	)
 	(segment
@@
 		(width 0.2)
 		(layer "In2.Cu")
+		(net 13)
+	)
+	(segment
+		(start 163.1 111.4)
+		(end 163.5 111)
+		(width 0.2)
+		(layer "B.Cu")
+		(net 23)
+	)
+	(segment
+		(start 157.24 111.4)
+		(end 163.1 111.4)
+		(width 0.2)
+		(layer "B.Cu")
+		(net 23)
+	)
+	(segment
+		(start 159 73.975)
+		(end 163.475 69.5)
+		(width 0.2)
+		(layer "F.Cu")
+		(net 24)
+	)
+	(segment
+		(start 157.24 93.62)
+		(end 159 91.86)
+		(width 0.2)
+		(layer "F.Cu")
+		(net 24)
+	)
+	(segment
+		(start 159 91.86)
+		(end 159 73.975)
+		(width 0.2)
+		(layer "F.Cu")
+		(net 24)
+	)
+	(segment
+		(start 157.24 93.62)
+		(end 160.5 96.88)
+		(width 0.2)
+		(layer "B.Cu")
+		(net 24)
+	)
+	(segment
+		(start 160.5 96.88)
+		(end 160.5 97.84)
+		(width 0.2)
+		(layer "B.Cu")
+		(net 24)
+	)
+	(segment
+		(start 160.5 97.84)
+		(end 163.5 100.84)
+		(width 0.2)
+		(layer "B.Cu")
 		(net 24)
 	)
