File: PCB_Glove.kicad_sch (KiCad schematic)
At the start: 12 parts, among them J1 HC-05, J2 MPU-9250/6500, J4 MPU-9250/6500, J5 FlexSensor_JST, J6 External_source, SW1 SW_SPST, SW2 SW_SPST, SW3 SW_SPST

Commit message: Polished Schematic
Connections:
- net +3V3: now reaches A1.17 (3V3), J4.7 (Pin_7)
- net A0: now reaches A1.19 (A0), J5.1 (Pin_1), R3.1
- net SDA: now reaches A1.23 (SDA/A4), J2.4 (Pin_4), J4.4 (Pin_4)
- net SCL: now reaches A1.24 (SCL/A5), J2.3 (Pin_3), J4.3 (Pin_3)
- net +5V: now reaches A1.27 (+5V), J1.5 (Pin_5), J2.1 (Pin_1), J4.1 (Pin_1), J5.2 (Pin_2)
- net INT1: now reaches A1.5 (D2), J2.8 (Pin_8)
- net INT2: now reaches A1.6 (D3), J4.8 (Pin_8)
- net VCC renamed +9V
Other:
- note added: "RX Bluetooth"
- note added: "TX Bluetooth"
- note removed: "+9V DC"
- note removed: "GND"
- note removed: "INT pin"
- note removed: "Vcc"
- title: Glove_Interface -> A_Glove_Interface
- moved on the sheet: J5, J6, SW1
